Commit message: Add some example nullspace tasks (#2)

File: models/ur_description/urdf/ur5_joint_limited_robot.urdf (robot description, URDF)
Before this commit: robot ur5, 11 links, 10 joints
Joints:
- joint elbow_joint: limit lower=-3.14159265359 upper=3.14159265359 effort=150.0 velocity=3.15 -> lower=-1.5707 upper=1.5707 effort=150.0 velocity=3.15
- joint shoulder_lift_joint: limit lower=-3.14159265359 upper=3.14159265359 effort=150.0 velocity=3.15 -> lower=-1.5707 upper=1.5707 effort=150.0 velocity=3.15
- joint wrist_1_joint: limit lower=-3.14159265359 upper=3.14159265359 effort=28.0 velocity=3.2 -> lower=-1.5707 upper=1.5707 effort=28.0 velocity=3.2
- joint wrist_2_joint: limit lower=-3.14159265359 upper=3.14159265359 effort=28.0 velocity=3.2 -> lower=-1.5707 upper=1.5707 effort=28.0 velocity=3.2
